File: mist-eeg/power.sch (KiCad schematic (older format))
At the start: 20 parts, among them J1 Power_5V-14V, Q1 20V @ 3A PMOS, U1 LTC2947, U2 LTC4412HV

Commit message: Hooked-up the SoM
Parts:
- renumbered TP11 to TP1, TP1 to TP2
Other:
- note added: "Power LED?"
Changed lines of the file:
@@
 	9150 2400 9100 2400
 $Comp
-L Connector:TestPoint TP1
+L Connector:TestPoint TP2
 U 1 1 60EA9E7A
 P 8700 2400
-F 0 "TP1" H 8700 2725 50  0000 C CNN
+F 0 "TP2" H 8700 2725 50  0000 C CNN
 F 1 "EXT_IN" H 8700 2634 50  0000 C CNN
 F 2 "TestPoint:TestPoint_Pad_D1.0mm" H 8900 2400 50  0001 C CNN
@@
 	8550 4700 8500 4700
 $Comp
-L Connector:TestPoint TP11
+L Connector:TestPoint TP1
 U 1 1 61425A62
 P 7300 5900
-F 0 "TP11" V 7254 6088 50  0000 L CNN
+F 0 "TP1" V 7254 6088 50  0000 L CNN
 F 1 "Power OK" V 7345 6088 50  0000 L CNN
 F 2 "" H 7500 5900 50  0001 C CNN
@@
 	0    1    1    0
 $EndComp
+Text Notes 8250 5800 0    50   ~ 0
+Power LED?
 $EndSCHEMATC

Commit message: Finish schematic and create interface specifications
Parts:
- removed TP1: Power OK, symbol Connector:TestPoint
- added D2: ON, LED_THT:LED_D3.0mm, symbol Device:LED
- added Q1: NMOS_DGS (5V), Package_TO_SOT_SMD:SOT-23, symbol Device:Q_NMOS_DGS
- added R6: 4k7, Resistor_SMD:R_0201_0603Metric, symbol Device:R_Small
- added R7: 1k, Resistor_SMD:R_0402_1005Metric, symbol Device:R_Small
- R4: footprint (none) -> Resistor_SMD:R_0201_0603Metric
- renumbered Q1 to Q2, R6 to R8, TP2 to TP1
Connections:
- net labels added: PG
- wire segments 105 -> 113
Other:
- note removed: "Power LED?"
Changed lines of the file:
@@
 	7850 2600 7900 2600
 $Comp
-L Device:R_Small R6
+L Device:R_Small R8
 U 1 1 60E9A912
 P 9000 2400
-F 0 "R6" V 8804 2400 50  0000 C CNN
+F 0 "R8" V 8804 2400 50  0000 C CNN
 F 1 "4k7" V 8895 2400 50  0000 C CNN
 F 2 "Resistor_SMD:R_0201_0603Metric" H 9000 2400 50  0001 C CNN
@@
 	9150 2400 9100 2400
 $Comp
-L Connector:TestPoint TP2
+L Connector:TestPoint TP1
 U 1 1 60EA9E7A
 P 8700 2400
-F 0 "TP2" H 8700 2725 50  0000 C CNN
+F 0 "TP1" H 8700 2725 50  0000 C CNN
 F 1 "EXT_IN" H 8700 2634 50  0000 C CNN
 F 2 "TestPoint:TestPoint_Pad_D1.0mm" H 8900 2400 50  0001 C CNN
@@
 +EXT_IN
 $Comp
-L Device:Q_PMOS_GDS Q1
+L Device:Q_PMOS_GDS Q2
 U 1 1 60EB8825
 P 8900 2750
-F 0 "Q1" V 9149 2750 50  0000 C CNN
+F 0 "Q2" V 9149 2750 50  0000 C CNN
 F 1 "20V @ 3A PMOS" V 9240 2750 50  0000 C CNN
 F 2 "Package_TO_SOT_SMD:TO-252-3_TabPin2" H 9100 2850 50  0001 C CNN
@@
 $EndComp
 $Comp
-L power:+3V3 #PWR013
+L power:+3V3 #PWR014
 U 1 1 61175ADA
 P 9150 2400
-F 0 "#PWR013" H 9150 2250 50  0001 C CNN
+F 0 "#PWR014" H 9150 2250 50  0001 C CNN
 F 1 "+3V3" V 9165 2528 50  0000 L CNN
 F 2 "" H 9150 2400 50  0001 C CNN
@@
 F 0 "R4" V 6304 5300 50  0000 C CNN
 F 1 "4k7" V 6395 5300 50  0000 C CNN
-F 2 "" H 6200 5300 50  0001 C CNN
+F 2 "Resistor_SMD:R_0201_0603Metric" H 6200 5300 50  0001 C CNN
 F 3 "~" H 6200 5300 50  0001 C CNN
 	1    6200 5300
@@
 Text Notes 1750 5200 0    50   ~ 10
 Rails
-Text Label 8500 4700 2    50   ~ 0
+Text Label 8800 4200 2    50   ~ 0
 STAGE_2
-Text HLabel 8550 4700 2    50   Output ~ 0
+Text HLabel 8850 4200 2    50   Output ~ 0
 AUDIO_OK
 Wire Wire Line
-	8550 4700 8500 4700
-$Comp
-L Connector:TestPoint TP1
-U 1 1 61425A62
-P 7300 5900
-F 0 "TP1" V 7254 6088 50  0000 L CNN
-F 1 "Power OK" V 7345 6088 50  0000 L CNN
-F 2 "" H 7500 5900 50  0001 C CNN
-F 3 "~" H 7500 5900 50  0001 C CNN
-	1    7300 5900
-	0    1    1    0
-$EndComp
-Text Notes 8250 5800 0    50   ~ 0
-Power LED?
+	8850 4200 8800 4200
+Text Label 7300 5900 0    50   ~ 0
+PG
+Text Label 8550 5350 2    50   ~ 0
+PG
+$Comp
+L Device:LED D2
+U 1 1 612ED13D
+P 8950 6000
+F 0 "D2" V 8989 5882 50  0000 R CNN
+F 1 "ON" V 8898 5882 50  0000 R CNN
+F 2 "LED_THT:LED_D3.0mm" H 8950 6000 50  0001 C CNN
+F 3 "~" H 8950 6000 50  0001 C CNN
+	1    8950 6000
+	0    -1   -1   0
+$EndComp
+$Comp
+L power:GND #PWR013
+U 1 1 612F0DA2
+P 8950 6200
+F 0 "#PWR013" H 8950 5950 50  0001 C CNN
+F 1 "GND" H 8955 6027 50  0000 C CNN
+F 2 "" H 8950 6200 50  0001 C CNN
+F 3 "" H 8950 6200 50  0001 C CNN
+	1    8950 6200
+	1    0    0    -1
+$EndComp
+Wire Wire Line
+	8950 6150 8950 6200
+$Comp
+L Device:Q_NMOS_DGS Q1
+U 1 1 612F7FA5
+P 8850 5350
+F 0 "Q1" H 9054 5396 50  0000 L CNN
+F 1 "NMOS_DGS (5V)" H 9054 5305 50  0000 L CNN
+F 2 "Package_TO_SOT_SMD:SOT-23" H 9050 5450 50  0001 C CNN
+F 3 "~" H 8850 5350 50  0001 C CNN
+	1    8850 5350
+	1    0    0    -1
+$EndComp
+Wire Wire Line
+	8950 5850 8950 5800
+Wire Wire Line
+	8950 5600 8950 5550
+Text HLabel 8950 5100 1    50   Input ~ 0
++5V_SOM
+Wire Wire Line
+	8950 5100 8950 5150
+$Comp
+L Device:R_Small R6
+U 1 1 6131A811
+P 8600 5200
+F 0 "R6" H 8541 5154 50  0000 R CNN
+F 1 "4k7" H 8541 5245 50  0000 R CNN
+F 2 "Resistor_SMD:R_0201_0603Metric" H 8600 5200 50  0001 C CNN
+F 3 "~" H 8600 5200 50  0001 C CNN
+	1    8600 5200
+	-1   0    0    1
+$EndComp
+Wire Wire Line
+	8550 5350 8600 5350
+Wire Wire Line
+	8600 5350 8600 5300
+Connection ~ 8600 5350
+Wire Wire Line
+	8600 5350 8650 5350
+Text HLabel 8600 5050 1    50   Input ~ 0
++5V_SOM
+Wire Wire Line
+	8600 5050 8600 5100
+$Comp
+L Device:R_Small R?
+U 1 1 613287EB
+P 8950 5700
+AR Path="/60D119DF/613287EB" Ref="R?"  Part="1"
+AR Path="/609A79EB/613287EB" Ref="R7"  Part="1"
+F 0 "R7" V 9054 5700 50  0000 C CNN
+F 1 "1k" V 9145 5700 50  0000 C CNN
+F 2 "Resistor_SMD:R_0402_1005Metric" H 8950 5700 50  0001 C CNN
+F 3 "~" H 8950 5700 50  0001 C CNN
+	1    8950 5700
+	1    0    0    -1
+$EndComp
 $EndSCHEMATC

Commit message: Advance routing
Parts:
- removed Q2: 20V @ 3A PMOS, Package_TO_SOT_SMD:TO-252-3_TabPin2, symbol Device:Q_PMOS_GDS
- removed TP1: EXT_IN, TestPoint:TestPoint_Pad_D1.0mm, symbol Connector:TestPoint
- removed U2: LTC4412HV, Package_TO_SOT_SMD:SOT-23-6, symbol components:LTC4412HV
- R8: value 4k7 -> DNF; footprint Resistor_SMD:R_0201_0603Metric -> Resistor_SMD:R_1206_3216Metric
Connections:
- net labels added: +3V3_SD
- net labels removed: +EXT_IN, ~ENA_EXT~
- wire segments 113 -> 97
Other:
- note added: "HWMon bypass"
- note removed: "5V @ 2A\nIntegrated ideal diode"
- note removed: "USB power"
Changed lines of the file:
@@
 $Descr USLetter 11000 8500
 encoding utf-8
-Sheet 2 12
+Sheet 2 11
 Title "Portiloop"
 Date "2021-06-07"
@@
 $EndDescr
 Text HLabel 7300 4450 2    50   Output ~ 0
-+3V3
++3V3_SD
 Text Notes 1750 5950 0    50   ~ 0
 3V3 V @ 1.75 A (TPS84A20):\n - SD card, 2.88 W max\n\n5V0 (clean) @ 50 mA:\n - ADS1299 Analog supply\n - LTC2947 supply\n\n1V8 (clean) @ 10 mA\n - ADAU1777 Analog supply
@@
 Text HLabel 3150 1500 2    50   Input ~ 0
 PWR_SCL
-$Sheet
-S 1450 2650 600  400
-U 60EAD252
-F0 "USB" 50
-F1 "USB.sch" 50
-F2 "+VSYS" O R 2050 2750 50
-F3 "SCL" I R 2050 2850 50
-F4 "SDA" B R 2050 2950 50
-F5 "~IRQ~" O L 1450 2750 50
-F6 "RST" I L 1450 2850 50
-F7 "ENA" O L 1450 2950 50
-$EndSheet
 $Comp
 L Connector:Screw_Terminal_01x02 J1
@@
 	-1   0    0    1
 $EndComp
-Wire Wire Line
-	7400 2550 7400 2500
-Text Notes 2800 2950 0    50   ~ 0
-5V @ 2A\nIntegrated ideal diode
 Text Notes 5650 2500 2    50   ~ 0
 5V - 14V @ 10W
@@
 	500  2500 4550 2500
 $Comp
-L components:LTC4412HV U2
-U 1 1 60E63456
-P 8250 2500
-F 0 "U2" H 8250 2825 50  0000 C CNN
-F 1 "LTC4412HV" H 8250 2734 50  0000 C CNN
-F 2 "Package_TO_SOT_SMD:SOT-23-6" H 8200 2400 50  0001 C CNN
-F 3 "" H 8200 2400 50  0001 C CNN
-	1    8250 2500
-	1    0    0    -1
-$EndComp
-Text Label 1400 2950 2    50   ~ 0
-~ENA_EXT~
-Wire Wire Line
-	1400 2950 1450 2950
-Text HLabel 2100 2950 2    50   BiDi ~ 0
-PWR_SDA
-Wire Wire Line
-	2100 2950 2050 2950
-Text HLabel 2100 2850 2    50   Input ~ 0
-PWR_SCL
-Wire Wire Line
-	2100 2850 2050 2850
-Wire Wire Line
-	7900 2500 7400 2500
-Text Label 7850 2600 2    50   ~ 0
-~ENA_EXT~
-Wire Wire Line
-	7850 2600 7900 2600
-$Comp
-L Device:R_Small R8
-U 1 1 60E9A912
-P 9000 2400
-F 0 "R8" V 8804 2400 50  0000 C CNN
-F 1 "4k7" V 8895 2400 50  0000 C CNN
-F 2 "Resistor_SMD:R_0201_0603Metric" H 9000 2400 50  0001 C CNN
-F 3 "~" H 9000 2400 50  0001 C CNN
-	1    9000 2400
-	0    1    1    0
-$EndComp
-Wire Wire Line
-	9150 2400 9100 2400
-$Comp
-L Connector:TestPoint TP1
-U 1 1 60EA9E7A
-P 8700 2400
-F 0 "TP1" H 8700 2725 50  0000 C CNN
-F 1 "EXT_IN" H 8700 2634 50  0000 C CNN
-F 2 "TestPoint:TestPoint_Pad_D1.0mm" H 8900 2400 50  0001 C CNN
-F 3 "~" H 8900 2400 50  0001 C CNN
-	1    8700 2400
-	1    0    0    -1
-$EndComp
-Wire Wire Line
-	8600 2400 8700 2400
-Text Label 2100 2750 0    50   ~ 0
-+PWR_IN
-Wire Wire Line
-	2100 2750 2050 2750
-Wire Wire Line
-	8700 2400 8900 2400
-Connection ~ 8700 2400
-$Comp
 L Device:D_TVS D?
 U 1 1 60ED35C5
@@
 	6400 2750 6400 2800
 Text Label 6600 2450 0    50   ~ 0
-+EXT_IN
-Wire Wire Line
-	6000 2600 6000 2550
++PWR_IN
 Wire Wire Line
 	6000 2550 5950 2550
-Text Label 7850 2400 2    50   ~ 0
-+EXT_IN
-Wire Wire Line
-	7850 2400 7900 2400
-Text Label 8600 2850 2    50   ~ 0
-+PWR_IN
-Wire Wire Line
-	8650 2600 8600 2600
-Text Label 9150 2850 0    50   ~ 0
-+EXT_IN
-$Comp
-L Device:Q_PMOS_GDS Q2
-U 1 1 60EB8825
-P 8900 2750
-F 0 "Q2" V 9149 2750 50  0000 C CNN
-F 1 "20V @ 3A PMOS" V 9240 2750 50  0000 C CNN
-F 2 "Package_TO_SOT_SMD:TO-252-3_TabPin2" H 9100 2850 50  0001 C CNN
-F 3 "~" H 8900 2750 50  0001 C CNN
-	1    8900 2750
-	0    1    1    0
-$EndComp
-Wire Wire Line
-	8900 2500 8900 2550
-Wire Wire Line
-	8600 2500 8900 2500
-Wire Wire Line
-	8700 2850 8650 2850
-Connection ~ 8650 2850
-Wire Wire Line
-	8650 2850 8650 2600
-Wire Wire Line
-	9150 2850 9100 2850
-Wire Wire Line
-	8600 2850 8650 2850
 Text Notes 500  3300 0    50   ~ 10
-USB power
+HWMon bypass
 Wire Notes Line
 	500  3300 10500 3300
@@
 F2 "OK" O R 7250 4600 50
 F3 "+PWR" I L 6450 4450 50
-F4 "+3V3" O R 7250 4450 50
+F4 "+3V3_SD" O R 7250 4450 50
 $EndSheet
 Text Label 6400 4450 2    50   ~ 0
@@
 $EndComp
 $Comp
-L power:GND #PWR012
-U 1 1 610A975E
-P 7400 2550
-F 0 "#PWR012" H 7400 2300 50  0001 C CNN
-F 1 "GND" H 7405 2377 50  0000 C CNN
-F 2 "" H 7400 2550 50  0001 C CNN
-F 3 "" H 7400 2550 50  0001 C CNN
-	1    7400 2550
-	1    0    0    -1
-$EndComp
-$Comp
 L power:GND #PWR09
 U 1 1 610A9BEC
@@
 F 3 "" H 1900 1700 50  0001 C CNN
 	1    1900 1700
-	0    1    1    0
-$EndComp
-$Comp
-L power:+3V3 #PWR014
-U 1 1 61175ADA
-P 9150 2400
-F 0 "#PWR014" H 9150 2250 50  0001 C CNN
-F 1 "+3V3" V 9165 2528 50  0000 L CNN
-F 2 "" H 9150 2400 50  0001 C CNN
-F 3 "" H 9150 2400 50  0001 C CNN
-	1    9150 2400
 	0    1    1    0
 $EndComp
@@
 Wire Wire Line
 	8950 5600 8950 5550
-Text HLabel 8950 5100 1    50   Input ~ 0
-+5V_SOM
 Wire Wire Line
 	8950 5100 8950 5150
@@
 Wire Wire Line
 	8600 5350 8650 5350
-Text HLabel 8600 5050 1    50   Input ~ 0
-+5V_SOM
 Wire Wire Line
 	8600 5050 8600 5100
@@
 	1    0    0    -1
 $EndComp
+Text Label 2100 2900 2    50   ~ 0
++PWR_IN
+Text Label 2500 2900 0    50   ~ 0
++PWR
+$Comp
+L Device:R_Small R8
+U 1 1 612F92EA
+P 2300 2900
+F 0 "R8" V 2104 2900 50  0000 C CNN
+F 1 "DNF" V 2195 2900 50  0000 C CNN
+F 2 "Resistor_SMD:R_1206_3216Metric" H 2300 2900 50  0001 C CNN
+F 3 "~" H 2300 2900 50  0001 C CNN
+	1    2300 2900
+	0    1    1    0
+$EndComp
+Wire Wire Line
+	2100 2900 2200 2900
+Wire Wire Line
+	2400 2900 2500 2900
+Wire Wire Line
+	6000 2600 6000 2550
+$Comp
+L power:+3V3 #PWR0139
+U 1 1 611097F5
+P 8600 5050
+F 0 "#PWR0139" H 8600 4900 50  0001 C CNN
+F 1 "+3V3" H 8615 5223 50  0000 C CNN
+F 2 "" H 8600 5050 50  0001 C CNN
+F 3 "" H 8600 5050 50  0001 C CNN
+	1    8600 5050
+	1    0    0    -1
+$EndComp
+$Comp
+L power:+3V3 #PWR0140
+U 1 1 61109884
+P 8950 5100
+F 0 "#PWR0140" H 8950 4950 50  0001 C CNN
+F 1 "+3V3" H 8965 5273 50  0000 C CNN
+F 2 "" H 8950 5100 50  0001 C CNN
+F 3 "" H 8950 5100 50  0001 C CNN
+	1    8950 5100
+	1    0    0    -1
+$EndComp

Commit message: Validation & fabrication layer
Parts:
- added R10, R9: 4k7, Resistor_SMD:R_0201_0603Metric, symbol Device:R_Small
- D1: symbol Device:D_TVS -> Diode:SM6T6V8A
- Q1: value NMOS_DGS (5V) -> NMOS_DGS (3V3)
Connections:
- wire segments 97 -> 101
Other:
- note added: "3V3 V @ 1.75 A (TPS63070):\n - SD card, 2.88 W max\n\n5V0 (clean) @ 50 mA:\n - ADS1299 Analog supply\n - LTC2947 supply\n\n1V8 (clean) @ 10 mA:\n - ADAU1777 Analog supply\n\n5V25 (intermediate) @ 100 mA:\n - clean voltage buck-boost\n\n5V @ 1.2 A:\n - SoM core voltage"
- note added: "ADC supplies:\n 1 - 5V25 (intermediate)\n 2 - 5V & 1V8 (clean)\n\nAudio:\n 1 - 1.8V (clean)\n 2 - 3.3V\n\nGlobal:\n 1 - 5.25V (Intermediate)\n 2 - 1.8V (Clean), 5V (Clean)\n 3 - 3.3V, 5V (Board power)"
- note removed: "3V3 V @ 1.75 A (TPS84A20):\n - SD card, 2.88 W max\n\n5V0 (clean) @ 50 mA:\n - ADS1299 Analog supply\n - LTC2947 supply\n\n1V8 (clean) @ 10 mA\n - ADAU1777 Analog supply"
- note removed: "ADC supplies:\n 1 - 5V25 (intermediate)\n 2 - 5V & 1V8 (clean)\n\nAudio:\n 1 - 1.8V (clean)\n 2 - 3.3V\n\nGlobal:\n 1 - 3.3V, 5.25V (Intermediate)\n 2 - 1.8V (Clean), 5V (Clean)\n 3 - 5V (Board power)"
- moved on the sheet: D2, Q1, R6, R7
Changed lines of the file:
@@
 Text HLabel 7300 4450 2    50   Output ~ 0
 +3V3_SD
-Text Notes 1750 5950 0    50   ~ 0
-3V3 V @ 1.75 A (TPS84A20):\n - SD card, 2.88 W max\n\n5V0 (clean) @ 50 mA:\n - ADS1299 Analog supply\n - LTC2947 supply\n\n1V8 (clean) @ 10 mA\n - ADAU1777 Analog supply
+Text Notes 1750 5350 0    50   ~ 0
+3V3 V @ 1.75 A (TPS63070):\n - SD card, 2.88 W max\n\n5V0 (clean) @ 50 mA:\n - ADS1299 Analog supply\n - LTC2947 supply\n\n1V8 (clean) @ 10 mA:\n - ADAU1777 Analog supply\n\n5V25 (intermediate) @ 100 mA:\n - clean voltage buck-boost\n\n5V @ 1.2 A:\n - SoM core voltage
 Text HLabel 7300 5000 2    50   Output ~ 0
 +5V0_ANA
@@
 Wire Notes Line
 	500  2500 4550 2500
-$Comp
-L Device:D_TVS D?
-U 1 1 60ED35C5
-P 6400 2600
-AR Path="/609A79EB/60EAD252/60ED35C5" Ref="D?"  Part="1"
-AR Path="/609A79EB/60ED35C5" Ref="D1"  Part="1"
-F 0 "D1" V 6446 2520 50  0000 R CNN
-F 1 "D_TVS" V 6355 2520 50  0000 R CNN
-F 2 "Diode_SMD:D_SMA" H 6400 2600 50  0001 C CNN
-F 3 "~" H 6400 2600 50  0001 C CNN
-	1    6400 2600
-	0    -1   -1   0
-$EndComp
 Wire Wire Line
 	6400 2750 6400 2800
@@
 Wire Notes Line
 	4550 500  4550 8000
-Text Notes 1750 6200 0    50   ~ 10
+Text Notes 1750 5600 0    50   ~ 10
 Sequencing
-Text Notes 1750 7200 0    50   ~ 0
-ADC supplies:\n 1 - 5V25 (intermediate)\n 2 - 5V & 1V8 (clean)\n\nAudio:\n 1 - 1.8V (clean)\n 2 - 3.3V\n\nGlobal:\n 1 - 3.3V, 5.25V (Intermediate)\n 2 - 1.8V (Clean), 5V (Clean)\n 3 - 5V (Board power)
+Text Notes 1750 6600 0    50   ~ 0
+ADC supplies:\n 1 - 5V25 (intermediate)\n 2 - 5V & 1V8 (clean)\n\nAudio:\n 1 - 1.8V (clean)\n 2 - 3.3V\n\nGlobal:\n 1 - 5.25V (Intermediate)\n 2 - 1.8V (Clean), 5V (Clean)\n 3 - 3.3V, 5V (Board power)
 $Sheet
 S 6450 3800 800  350
@@
 F3 "+PWR" I L 6450 3900 50
 F4 "+5V25" O R 7250 3900 50
+F5 "ENA" I L 6450 4000 50
 $EndSheet
 Text Label 6400 3900 2    50   ~ 0
@@
 F3 "+PWR" I L 6450 4450 50
 F4 "+3V3_SD" O R 7250 4450 50
+F5 "ENA" I L 6450 4550 50
 $EndSheet
 Text Label 6400 4450 2    50   ~ 0
@@
 Wire Wire Line
 	5950 2450 6100 2450
-Wire Wire Line
-	6400 2450 6550 2450
-Wire Wire Line
-	6300 2450 6400 2450
-Connection ~ 6400 2450
 $Comp
 L power:GND #PWR06
@@
 Wire Wire Line
 	7300 5800 7250 5800
-Text Notes 1750 5200 0    50   ~ 10
+Text Notes 1750 4100 0    50   ~ 10
 Rails
 Text Label 8800 4200 2    50   ~ 0
@@
 Text Label 7300 5900 0    50   ~ 0
 PG
-Text Label 8550 5350 2    50   ~ 0
+Text Label 8800 5950 2    50   ~ 0
 PG
 $Comp
 L Device:LED D2
 U 1 1 612ED13D
-P 8950 6000
-F 0 "D2" V 8989 5882 50  0000 R CNN
-F 1 "ON" V 8898 5882 50  0000 R CNN
-F 2 "LED_THT:LED_D3.0mm" H 8950 6000 50  0001 C CNN
-F 3 "~" H 8950 6000 50  0001 C CNN
-	1    8950 6000
+P 9200 5550
+F 0 "D2" V 9239 5432 50  0000 R CNN
+F 1 "ON" V 9148 5432 50  0000 R CNN
+F 2 "LED_THT:LED_D3.0mm" H 9200 5550 50  0001 C CNN
+F 3 "~" H 9200 5550 50  0001 C CNN
+	1    9200 5550
 	0    -1   -1   0
 $EndComp
@@
 L power:GND #PWR013
 U 1 1 612F0DA2
-P 8950 6200
-F 0 "#PWR013" H 8950 5950 50  0001 C CNN
-F 1 "GND" H 8955 6027 50  0000 C CNN
-F 2 "" H 8950 6200 50  0001 C CNN
-F 3 "" H 8950 6200 50  0001 C CNN
-	1    8950 6200
+P 9200 6200
+F 0 "#PWR013" H 9200 5950 50  0001 C CNN
+F 1 "GND" H 9205 6027 50  0000 C CNN
+F 2 "" H 9200 6200 50  0001 C CNN
+F 3 "" H 9200 6200 50  0001 C CNN
+	1    9200 6200
 	1    0    0    -1
 $EndComp
-Wire Wire Line
-	8950 6150 8950 6200
 $Comp
 L Device:Q_NMOS_DGS Q1
 U 1 1 612F7FA5
-P 8850 5350
-F 0 "Q1" H 9054 5396 50  0000 L CNN
-F 1 "NMOS_DGS (5V)" H 9054 5305 50  0000 L CNN
-F 2 "Package_TO_SOT_SMD:SOT-23" H 9050 5450 50  0001 C CNN
-F 3 "~" H 8850 5350 50  0001 C CNN
-	1    8850 5350
+P 9100 5950
+F 0 "Q1" H 9304 5996 50  0000 L CNN
+F 1 "NMOS_DGS (3V3)" H 9304 5905 50  0000 L CNN
+F 2 "Package_TO_SOT_SMD:SOT-23" H 9300 6050 50  0001 C CNN
+F 3 "~" H 9100 5950 50  0001 C CNN
+	1    9100 5950
 	1    0    0    -1
 $EndComp
 Wire Wire Line
-	8950 5850 8950 5800
-Wire Wire Line
-	8950 5600 8950 5550
-Wire Wire Line
-	8950 5100 8950 5150
+	9200 5400 9200 5350
+Wire Wire Line
+	9200 6200 9200 6150
+Wire Wire Line
+	9200 5100 9200 5150
 $Comp
 L Device:R_Small R6
 U 1 1 6131A811
-P 8600 5200
-F 0 "R6" H 8541 5154 50  0000 R CNN
-F 1 "4k7" H 8541 5245 50  0000 R CNN
-F 2 "Resistor_SMD:R_0201_0603Metric" H 8600 5200 50  0001 C CNN
-F 3 "~" H 8600 5200 50  0001 C CNN
-	1    8600 5200
+P 8850 5800
+F 0 "R6" H 8791 5754 50  0000 R CNN
+F 1 "4k7" H 8791 5845 50  0000 R CNN
+F 2 "Resistor_SMD:R_0201_0603Metric" H 8850 5800 50  0001 C CNN
+F 3 "~" H 8850 5800 50  0001 C CNN
+	1    8850 5800
 	-1   0    0    1
 $EndComp
 Wire Wire Line
-	8550 5350 8600 5350
-Wire Wire Line
-	8600 5350 8600 5300
-Connection ~ 8600 5350
-Wire Wire Line
-	8600 5350 8650 5350
-Wire Wire Line
-	8600 5050 8600 5100
+	8800 5950 8850 5950
+Wire Wire Line
+	8850 5950 8850 5900
+Connection ~ 8850 5950
+Wire Wire Line
+	8850 5950 8900 5950
+Wire Wire Line
+	8850 5650 8850 5700
 $Comp
 L Device:R_Small R?
 U 1 1 613287EB
-P 8950 5700
+P 9200 5250
 AR Path="/60D119DF/613287EB" Ref="R?"  Part="1"
 AR Path="/609A79EB/613287EB" Ref="R7"  Part="1"
-F 0 "R7" V 9054 5700 50  0000 C CNN
-F 1 "1k" V 9145 5700 50  0000 C CNN
-F 2 "Resistor_SMD:R_0402_1005Metric" H 8950 5700 50  0001 C CNN
-F 3 "~" H 8950 5700 50  0001 C CNN
-	1    8950 5700
+F 0 "R7" V 9304 5250 50  0000 C CNN
+F 1 "1k" V 9395 5250 50  0000 C CNN
+F 2 "Resistor_SMD:R_0402_1005Metric" H 9200 5250 50  0001 C CNN
+F 3 "~" H 9200 5250 50  0001 C CNN
+	1    9200 5250
 	1    0    0    -1
 $EndComp
@@
 L power:+3V3 #PWR0139
 U 1 1 611097F5
-P 8600 5050
-F 0 "#PWR0139" H 8600 4900 50  0001 C CNN
-F 1 "+3V3" H 8615 5223 50  0000 C CNN
-F 2 "" H 8600 5050 50  0001 C CNN
-F 3 "" H 8600 5050 50  0001 C CNN
-	1    8600 5050
+P 8850 5650
+F 0 "#PWR0139" H 8850 5500 50  0001 C CNN
+F 1 "+3V3" H 8865 5823 50  0000 C CNN
+F 2 "" H 8850 5650 50  0001 C CNN
+F 3 "" H 8850 5650 50  0001 C CNN
+	1    8850 5650
 	1    0    0    -1
 $EndComp
@@
 L power:+3V3 #PWR0140
 U 1 1 61109884
-P 8950 5100
-F 0 "#PWR0140" H 8950 4950 50  0001 C CNN
-F 1 "+3V3" H 8965 5273 50  0000 C CNN
-F 2 "" H 8950 5100 50  0001 C CNN
-F 3 "" H 8950 5100 50  0001 C CNN
-	1    8950 5100
+P 9200 5100
+F 0 "#PWR0140" H 9200 4950 50  0001 C CNN
+F 1 "+3V3" H 9215 5273 50  0000 C CNN
+F 2 "" H 9200 5100 50  0001 C CNN
+F 3 "" H 9200 5100 50  0001 C CNN
+	1    9200 5100
 	1    0    0    -1
 $EndComp
+$Comp
+L Diode:SM6T6V8A D?
+U 1 1 60ED35C5
+P 6400 2600
+AR Path="/609A79EB/60EAD252/60ED35C5" Ref="D?"  Part="1"
+AR Path="/609A79EB/60ED35C5" Ref="D1"  Part="1"
+F 0 "D1" V 6446 2520 50  0000 R CNN
+F 1 "D_TVS" V 6355 2520 50  0000 R CNN
+F 2 "Diode_SMD:D_SMA" H 6400 2600 50  0001 C CNN
+F 3 "~" H 6400 2600 50  0001 C CNN
+	1    6400 2600
+	0    1    1    0
+$EndComp
+Wire Wire Line
+	6300 2450 6400 2450
+Connection ~ 6400 2450
+Wire Wire Line
+	6400 2450 6550 2450
+Wire Wire Line
+	9200 5700 9200 5750
+Text Label 6150 4550 2    50   ~ 0
+STAGE_2
+Wire Wire Line
+	6400 4550 6450 4550
+$Comp
+L Device:R_Small R?
+U 1 1 610D8759
+P 6300 4000
+AR Path="/609A79EB/60F89803/610D8759" Ref="R?"  Part="1"
+AR Path="/609A79EB/610D8759" Ref="R9"  Part="1"
+F 0 "R9" V 6404 4000 50  0000 C CNN
+F 1 "4k7" V 6495 4000 50  0000 C CNN
+F 2 "Resistor_SMD:R_0201_0603Metric" H 6300 4000 50  0001 C CNN
+F 3 "~" H 6300 4000 50  0001 C CNN
+	1    6300 4000
+	0    1    1    0
+$EndComp
+Wire Wire Line
+	6150 4000 6200 4000
+Wire Wire Line
+	6400 4000 6450 4000
+Text Label 6150 4000 2    50   ~ 0
++PWR
+$Comp
+L Device:R_Small R?
+U 1 1 610E9FA4
+P 6300 4550
+AR Path="/609A79EB/60F89803/610E9FA4" Ref="R?"  Part="1"
+AR Path="/609A79EB/610E9FA4" Ref="R10"  Part="1"
+F 0 "R10" V 6404 4550 50  0000 C CNN
+F 1 "4k7" V 6495 4550 50  0000 C CNN
+F 2 "Resistor_SMD:R_0201_0603Metric" H 6300 4550 50  0001 C CNN
+F 3 "~" H 6300 4550 50  0001 C CNN
+	1    6300 4550
+	0    1    1    0
+$EndComp
+Wire Wire Line
+	6150 4550 6200 4550
 $EndSCHEMATC

Commit message: Update footprints based upon piece availability & generate manufacturing files
Parts:
- F1: footprint Fuse:Fuse_1206_3216Metric_Pad1.42x1.75mm_HandSolder -> Fuse:Fuse_2920_7451Metric
Changed lines of the file:
@@
 F 0 "F1" V 5995 2450 50  0000 C CNN
 F 1 "3 A, 20 V" V 6086 2450 50  0000 C CNN
-F 2 "Fuse:Fuse_1206_3216Metric_Pad1.42x1.75mm_HandSolder" H 6250 2250 50  0001 L CNN
+F 2 "Fuse:Fuse_2920_7451Metric" H 6250 2250 50  0001 L CNN
 F 3 "~" H 6200 2450 50  0001 C CNN
 	1    6200 2450
