File: portiloop.kicad_sch (KiCad schematic)
At the start: 83 parts, among them J1-A1 SSQ-120-03-G-D, J2-R1 61301011021, Q1 IRLML2502, SW1 A6H-2102, U1 LT3042xMSE, U2 LT3042xMSE, U3 LM2662MX/NOPB, U4 LT3094xMSE, U5 ADS1299IPAG

Commit message: version v2.3 KiCad 9.0.6
Parts:
- removed D3: LTST-C190GKT, Portiloop:FP-LTST-C190GKT-MFG, symbol Portiloop:LTST-C190GKT
- removed R7: 1k, Portiloop:1608[0603]_res_3d, symbol Portiloop:1608[0603]_res
Connections:
- net GPIO4/LED is gone; now on an unnamed net: U5.46 (GPIO4)
- net at R8.1, U5.42 (GPIO1), U5.44 (GPIO2): now also U5.45 (GPIO3)
- net GPIO39/LEDCTL: now reaches J1-A1.40
- net GPIO39/LEDCTL: now also R6.1
- removed net GPIO3/LEDCTL: R6.1, U5.45 (GPIO3)
- no-connect marks 19 -> 40
Other:
- moved on the sheet: J1-A1, JMP1-R1, JMP2-R1, JMP3-R1, M1, M2, M3, M4, Q1, R5, R6
