File: portiloop.kicad_pcb (KiCad board)
At the start: 2 copper layers, 64 x 48 mm, 83 parts, among them J1-A1 SSQ-120-03-G-D, J2-R1 61301011021, Q1 IRLML2502, SW1 A6H-2102, U1 LT3042xMSE, U2 LT3042xMSE, U3 LM2662MX/NOPB, U4 LT3094xMSE, U5 ADS1299IPAG

Commit message: version v2.3 KiCad 9.0.6
Parts:
- removed D3: LTST-C190GKT, Portiloop:FP-LTST-C190GKT-MFG
- removed R7: 1k, Portiloop:1608[0603]_res_3d
Connections:
- J1-A1 pad 40: unconnected-(J1-A1-Pad40) -> /GPIO39/LEDCTL
- R6 pad 1: /GPIO3/LEDCTL -> /GPIO39/LEDCTL
- U5 pad 45: /GPIO3/LEDCTL -> Net-(U5A-GPIO1)
- U5 pad 46: /GPIO4/LED -> Net-(U5A-GPIO1)
Routing:
- net /GPIO39/LEDCTL: track 0.00 -> 80.5 mm, vias 0 -> 1
- net /GPIO4/LED: track 48.1 -> 0.00 mm, vias 2 -> 0
- net /GPIO3/LEDCTL: track 37.7 -> 0.00 mm, vias 2 -> 0
- net Net-(U5A-GPIO1): track 6.91 -> 13.2 mm
- net /MISO: track 36.3 -> 32.9 mm
- net /BiasOut: track 21.8 -> 23.8 mm
- net Net-(D3-A): track 1.81 -> 0.00 mm
- net +3.3V: track 43.8 -> 45.1 mm
- net /GPIO37: track 25.6 -> 26.5 mm
- net /LEDGNDCTL: track 54.2 -> 53.3 mm
- net /MOSI: track 38.4 -> 37.6 mm
- net /Ref: track 7.75 -> 8.42 mm
- net /START: track 39.7 -> 39.1 mm
- net GND: vias 22 -> 27

Commit message: version v2.3 KiCad 9.0.6
Routing:
- net GND: vias 27 -> 26
Other:
- board text added: "GPIO10:LED_B"
- board text added: "GPIO22:LED_R"
- board text added: "GPIO37:START"
- board text added: "GPIO39:LEDCTL"
- board text added: "GPIO9:LED_G"
- board text removed: "GPIO10/LED_B"
- board text removed: "GPIO22/LED_R"
- board text removed: "GPIO9/LED_G"

Commit message: version v2.3 KiCad 9.0.6
Routing:
- net -2V5: track 115.4 -> 114.3 mm
- net /GPIO39/LEDCTL: track 80.5 -> 81.6 mm
- net GND: track 377.4 -> 378.4 mm
- net /DRDY: track 46.7 -> 47.6 mm
